Commit message: fix joint names gazebo bug

File: i2rt/bimanual/rtop_description/urdf/yam_arm.xacro (robot description, xacro)
@@ -42,5 +42,5 @@
       </visual>
     </link>
-    <link name="${prefix}joint1">
+    <link name="${prefix}joint1_link">
       <inertial>
         <origin xyz="0.0 0.0 0.0" rpy="0.0 0.0 0.0"/>
@@ -51,5 +51,5 @@
     <joint type="revolute" name="${prefix}joint1">
       <parent link="${prefix}arm"/>
-      <child link="${prefix}joint1"/>
+      <child link="${prefix}joint1_link"/>
       <origin xyz="0.0 0.0 0.0631" rpy="0.0 0.0 1.5707963267948963"/>
       <axis xyz="0.0 0.0 1.0"/>
@@ -57,5 +57,5 @@
     </joint>
     <joint type="fixed" name="${prefix}joint1_offset">
-      <parent link="${prefix}joint1"/>
+      <parent link="${prefix}joint1_link"/>
       <child link="${prefix}link_1"/>
       <origin xyz="-0.0 -0.0 -0.0" rpy="0.0 0.0 0.0"/>
@@ -87,5 +87,5 @@
       </visual>
     </link>
-    <link name="${prefix}joint2">
+    <link name="${prefix}joint2_link">
       <inertial>
         <origin xyz="0.0 0.0 0.0" rpy="0.0 0.0 0.0"/>
@@ -96,5 +96,5 @@
     <joint type="revolute" name="${prefix}joint2">
       <parent link="${prefix}link_1"/>
-      <child link="${prefix}joint2"/>
+      <child link="${prefix}joint2_link"/>
       <origin xyz="2.5e-05 -0.02 0.0409" rpy="1.5707963267948966 0.0 1.5707963267948966"/>
       <axis xyz="0.0 0.0 1.0"/>
@@ -102,5 +102,5 @@
     </joint>
     <joint type="fixed" name="${prefix}joint2_offset">
-      <parent link="${prefix}joint2"/>
+      <parent link="${prefix}joint2_link"/>
       <child link="${prefix}link_2"/>
       <origin xyz="-0.0 -0.0 -0.0" rpy="0.0 0.0 0.0"/>
@@ -138,5 +138,5 @@
       </visual>
     </link>
-    <link name="${prefix}joint3">
+    <link name="${prefix}joint3_link">
       <inertial>
         <origin xyz="0.0 0.0 0.0" rpy="0.0 0.0 0.0"/>
@@ -147,5 +147,5 @@
     <joint type="revolute" name="${prefix}joint3">
       <parent link="${prefix}link_2"/>
-      <child link="${prefix}joint3"/>
+      <child link="${prefix}joint3_link"/>
       <origin xyz="0.264 0.0 0.0" rpy="3.141592653589793 0.0 0.0"/>
       <axis xyz="0.0 0.0 1.0"/>
@@ -153,5 +153,5 @@
     </joint>
     <joint type="fixed" name="${prefix}joint3_offset">
-      <parent link="${prefix}joint3"/>
+      <parent link="${prefix}joint3_link"/>
       <child link="${prefix}link_3"/>
       <origin xyz="-0.0 -0.0 -0.0" rpy="0.0 0.0 0.0"/>
@@ -171,5 +171,5 @@
       </visual>
     </link>
-    <link name="${prefix}joint4">
+    <link name="${prefix}joint4_link">
       <inertial>
         <origin xyz="0.0 0.0 0.0" rpy="0.0 0.0 0.0"/>
@@ -180,5 +180,5 @@
     <joint type="revolute" name="${prefix}joint4">
       <parent link="${prefix}link_3"/>
-      <child link="${prefix}joint4"/>
+      <child link="${prefix}joint4_link"/>
       <origin xyz="-0.245 -0.06 0.0" rpy="0.0 0.0 0.0"/>
       <axis xyz="0.0 0.0 1.0"/>
@@ -186,5 +186,5 @@
     </joint>
     <joint type="fixed" name="${prefix}joint4_offset">
-      <parent link="${prefix}joint4"/>
+      <parent link="${prefix}joint4_link"/>
       <child link="${prefix}link_4"/>
       <origin xyz="-0.0 -0.0 -0.0" rpy="0.0 0.0 0.0"/>
@@ -204,5 +204,5 @@
       </visual>
     </link>
-    <link name="${prefix}joint5">
+    <link name="${prefix}joint5_link">
       <inertial>
         <origin xyz="0.0 0.0 0.0" rpy="0.0 0.0 0.0"/>
@@ -213,5 +213,5 @@
     <joint type="revolute" name="${prefix}joint5">
       <parent link="${prefix}link_4"/>
-      <child link="${prefix}joint5"/>
+      <child link="${prefix}joint5_link"/>
       <origin xyz="-0.074 -0.0395 2.5e-05" rpy="-1.5707963267948966 1.5707963267948966 0.0"/>
       <axis xyz="0.0 0.0 1.0"/>
@@ -219,5 +219,5 @@
     </joint>
     <joint type="fixed" name="${prefix}joint5_offset">
-      <parent link="${prefix}joint5"/>
+      <parent link="${prefix}joint5_link"/>
       <child link="${prefix}link_5"/>
       <origin xyz="-0.0 -0.0 -0.0" rpy="0.0 0.0 0.0"/>
@@ -243,5 +243,5 @@
       </visual>
     </link>
-    <link name="${prefix}joint6">
+    <link name="${prefix}joint6_link">
       <inertial>
         <origin xyz="0.0 0.0 0.0" rpy="0.0 0.0 0.0"/>
@@ -252,5 +252,5 @@
     <joint type="revolute" name="${prefix}joint6">
       <parent link="${prefix}link_5"/>
-      <child link="${prefix}joint6"/>
+      <child link="${prefix}joint6_link"/>
       <origin xyz="0.0 0.0353 0.0395" rpy="-1.5707963267948963 0.0 0.0"/>
       <axis xyz="0.0 0.0 1.0"/>
@@ -258,5 +258,5 @@
     </joint>
     <joint type="fixed" name="${prefix}joint6_offset">
-      <parent link="${prefix}joint6"/>
+      <parent link="${prefix}joint6_link"/>
       <child link="${prefix}link_6"/>
       <origin xyz="-0.0 -0.0 -0.0" rpy="0.0 0.0 0.0"/>
@@ -282,5 +282,5 @@
       </visual>
     </link>
-    <link name="${prefix}left_finger">
+    <link name="${prefix}left_finger_link">
       <inertial>
         <origin xyz="0.0 0.0 0.0" rpy="0.0 0.0 0.0"/>
@@ -291,5 +291,5 @@
     <joint type="prismatic" name="${prefix}left_finger">
       <parent link="${prefix}link_6"/>
-      <child link="${prefix}left_finger"/>
+      <child link="${prefix}left_finger_link"/>
       <origin xyz="-0.037 0.0392 0.0605" rpy="-0.0 1.5707963267948966 0.0"/>
       <axis xyz="0.0 0.0 1.0"/>
@@ -297,5 +297,5 @@
     </joint>
     <joint type="fixed" name="${prefix}left_finger_offset">
-      <parent link="${prefix}left_finger"/>
+      <parent link="${prefix}left_finger_link"/>
       <child link="${prefix}link_left_finger"/>
       <origin xyz="-0.0 -0.0 -0.0" rpy="0.0 0.0 0.0"/>
@@ -345,5 +345,5 @@
       </visual>
     </link>
-    <link name="${prefix}right_finger">
+    <link name="${prefix}right_finger_link">
       <inertial>
         <origin xyz="0.0 0.0 0.0" rpy="0.0 0.0 0.0"/>
@@ -354,5 +354,5 @@
     <joint type="prismatic" name="${prefix}right_finger">
       <parent link="${prefix}link_6"/>
-      <child link="${prefix}right_finger"/>
+      <child link="${prefix}right_finger_link"/>
       <origin xyz="0.037 -0.0392 0.0605" rpy="-0.0 1.5707963267948966 0.0"/>
       <axis xyz="0.0 0.0 1.0"/>
@@ -360,5 +360,5 @@
     </joint>
     <joint type="fixed" name="${prefix}right_finger_offset">
-      <parent link="${prefix}right_finger"/>
+      <parent link="${prefix}right_finger_link"/>
       <child link="${prefix}link_right_finger"/>
       <origin xyz="-0.0 -0.0 -0.0" rpy="0.0 0.0 0.0"/>
