Commit message: reorder simplify xacro

File: i2rt/bimanual/rtop_description/urdf/rtop.urdf.xacro (robot description, xacro)
@@ -1,6 +1,6 @@
 <?xml version="1.0"?>
 <robot xmlns:xacro="http://www.ros.org/wiki/xacro" name="rtop">
-  <!-- Include the arm macro -->
-  <xacro:include filename="yam_arm.xacro"/>
+  <!-- Include the arm macro from yam_arm_description -->
+  <xacro:include filename="$(find yam_arm_description)/urdf/yam_arm_macro.xacro"/>
   <!-- Base link (body) -->
   <link name="base">

File: i2rt/bimanual/rtop_description/urdf/rtop_gazebo.urdf.xacro (robot description, xacro)
@@ -8,8 +8,115 @@
   <!-- ROS2 Control for Gazebo -->
   <xacro:if value="$(arg use_gazebo)">
-    <xacro:include filename="$(find rtop_description)/urdf/gazebo_sim_ros2_control.urdf.xacro"/>
-    <xacro:load_gazebo_sim_ros2_control_plugin robot_name="rtop" ros2_controllers_path="$(arg ros2_controllers_path)" use_gazebo="$(arg use_gazebo)"/>
-    <xacro:include filename="$(find rtop_description)/urdf/ros2_control.urdf.xacro" />
-    <xacro:ros2_control_interfaces/>
+    <!-- Gazebo ROS2 Control Plugin -->
+    <gazebo>
+      <plugin filename="gz_ros2_control-system" name="gz_ros2_control::GazeboSimROS2ControlPlugin">
+        <parameters>$(arg ros2_controllers_path)</parameters>
+        <ros>
+          <remapping>/controller_manager/robot_description:=/robot_description</remapping>
+        </ros>
+      </plugin>
+    </gazebo>
+    <!-- ROS2 Control Interfaces -->
+    <ros2_control name="IgnitionSystem" type="system">
+      <hardware>
+        <plugin>gz_ros2_control/GazeboSimSystem</plugin>
+      </hardware>
+      <joint name="left_joint1">
+        <command_interface name="position"/>
+        <state_interface name="position" />
+        <state_interface name="velocity"/>
+        <state_interface name="effort"/>
+      </joint>
+      <joint name="left_joint2">
+        <command_interface name="position"/>
+        <state_interface name="position"/>
+        <state_interface name="velocity"/>
+        <state_interface name="effort"/>
+      </joint>
+      <joint name="left_joint3">
+        <command_interface name="position"/>
+        <state_interface name="position"/>
+        <state_interface name="velocity"/>
+        <state_interface name="effort"/>
+      </joint>
+      <joint name="left_joint4">
+        <command_interface name="position"/>
+        <state_interface name="position"/>
+        <state_interface name="velocity"/>
+        <state_interface name="effort"/>
+      </joint>
+      <joint name="left_joint5">
+        <command_interface name="position"/>
+        <state_interface name="position"/>
+        <state_interface name="velocity"/>
+        <state_interface name="effort"/>
+      </joint>
+      <joint name="left_joint6">
+        <command_interface name="position"/>
+        <state_interface name="position"/>
+        <state_interface name="velocity"/>
+        <state_interface name="effort"/>
+      </joint>
+      <joint name="left_left_finger">
+        <command_interface name="position"/>
+        <state_interface name="position"/>
+        <state_interface name="velocity"/>
+        <state_interface name="effort"/>
+      </joint>
+      <joint name="left_right_finger">
+        <command_interface name="position"/>
+        <state_interface name="position"/>
+        <state_interface name="velocity"/>
+        <state_interface name="effort"/>
+      </joint>
+      <joint name="right_joint1">
+        <command_interface name="position"/>
+        <state_interface name="position" />
+        <state_interface name="velocity"/>
+        <state_interface name="effort"/>
+      </joint>
+      <joint name="right_joint2">
+        <command_interface name="position"/>
+        <state_interface name="position"/>
+        <state_interface name="velocity"/>
+        <state_interface name="effort"/>
+      </joint>
+      <joint name="right_joint3">
+        <command_interface name="position"/>
+        <state_interface name="position"/>
+        <state_interface name="velocity"/>
+        <state_interface name="effort"/>
+      </joint>
+      <joint name="right_joint4">
+        <command_interface name="position"/>
+        <state_interface name="position"/>
+        <state_interface name="velocity"/>
+        <state_interface name="effort"/>
+      </joint>
+      <joint name="right_joint5">
+        <command_interface name="position"/>
+        <state_interface name="position"/>
+        <state_interface name="velocity"/>
+        <state_interface name="effort"/>
+      </joint>
+      <joint name="right_joint6">
+        <command_interface name="position"/>
+        <state_interface name="position"/>
+        <state_interface name="velocity"/>
+        <state_interface name="effort"/>
+      </joint>
+      <joint name="right_left_finger">
+        <command_interface name="position"/>
+        <state_interface name="position"/>
+        <state_interface name="velocity"/>
+        <state_interface name="effort"/>
+      </joint>
+      <joint name="right_right_finger">
+        <command_interface name="position"/>
+        <state_interface name="position"/>
+        <state_interface name="velocity"/>
+        <state_interface name="effort"/>
+      </joint>
+    </ros2_control>
   </xacro:if>
 </robot>
