Commit message: order code, gazebo launch, usd clean way

File: i2rt/bimanual/rtop_description/urdf/rtop.urdf (robot description, URDF)
Before this commit: robot rtop, 49 links, 48 joints
Links:
- removed link left_joint1
- removed link left_joint2
- removed link left_joint3
- removed link left_joint4
- removed link left_joint5
- removed link left_joint6
- removed link left_left_finger
- removed link left_right_finger
- removed link right_joint1
- removed link right_joint2
- removed link right_joint3
- removed link right_joint4
- removed link right_joint5
- removed link right_joint6
- removed link right_left_finger
- removed link right_right_finger
- added link left_joint1_link, mass 0.001
- added link left_joint2_link, mass 0.001
- added link left_joint3_link, mass 0.001
- added link left_joint4_link, mass 0.001
- added link left_joint5_link, mass 0.001
- added link left_joint6_link, mass 0.001
- added link left_left_finger_link, mass 0.001
- added link left_right_finger_link, mass 0.001
- added link right_joint1_link, mass 0.001
- added link right_joint2_link, mass 0.001
- added link right_joint3_link, mass 0.001
- added link right_joint4_link, mass 0.001
- added link right_joint5_link, mass 0.001
- added link right_joint6_link, mass 0.001
- added link right_left_finger_link, mass 0.001
- added link right_right_finger_link, mass 0.001
Joints:
- joint left_joint1: child left_joint1 -> left_joint1_link
- joint left_joint1_offset: parent left_joint1 -> left_joint1_link
- joint left_joint2: child left_joint2 -> left_joint2_link
- joint left_joint2_offset: parent left_joint2 -> left_joint2_link
- joint left_joint3: child left_joint3 -> left_joint3_link
- joint left_joint3_offset: parent left_joint3 -> left_joint3_link
- joint left_joint4: child left_joint4 -> left_joint4_link
- joint left_joint4_offset: parent left_joint4 -> left_joint4_link
- joint left_joint5: child left_joint5 -> left_joint5_link
- joint left_joint5_offset: parent left_joint5 -> left_joint5_link
- joint left_joint6: child left_joint6 -> left_joint6_link
- joint left_joint6_offset: parent left_joint6 -> left_joint6_link
- joint left_left_finger: child left_left_finger -> left_left_finger_link
- joint left_left_finger_offset: parent left_left_finger -> left_left_finger_link
- joint left_right_finger: child left_right_finger -> left_right_finger_link
- joint left_right_finger_offset: parent left_right_finger -> left_right_finger_link
- joint right_joint1: child right_joint1 -> right_joint1_link
- joint right_joint1_offset: parent right_joint1 -> right_joint1_link
- joint right_joint2: child right_joint2 -> right_joint2_link
- joint right_joint2_offset: parent right_joint2 -> right_joint2_link
- joint right_joint3: child right_joint3 -> right_joint3_link
- joint right_joint3_offset: parent right_joint3 -> right_joint3_link
- joint right_joint4: child right_joint4 -> right_joint4_link
- joint right_joint4_offset: parent right_joint4 -> right_joint4_link
- joint right_joint5: child right_joint5 -> right_joint5_link
- joint right_joint5_offset: parent right_joint5 -> right_joint5_link
- joint right_joint6: child right_joint6 -> right_joint6_link
- joint right_joint6_offset: parent right_joint6 -> right_joint6_link
- joint right_left_finger: child right_left_finger -> right_left_finger_link
- joint right_left_finger_offset: parent right_left_finger -> right_left_finger_link
- joint right_right_finger: child right_right_finger -> right_right_finger_link
- joint right_right_finger_offset: parent right_right_finger -> right_right_finger_link

File: i2rt/bimanual/rtop_moveit_config/config/rtop_calib.ros2_control.xacro (robot description, xacro)
@@ -8,6 +8,6 @@
                 <!-- plugin>mock_components/GenericSystem</plugin -->
                 <plugin>topic_based_ros2_control/TopicBasedSystem</plugin>
-                <param name="joint_commands_topic">/isaac_joint_command</param>
-                <param name="joint_states_topic">/isaac_joint_states</param>
+                <param name="joint_commands_topic">/joint_command</param>
+                <param name="joint_states_topic">/joint_states</param>
             </hardware>
             <!-- Left Arm Joints -->

File: i2rt/bimanual/rtop_moveit_config/config/rtop_calib.urdf.xacro (robot description, xacro)
@@ -3,5 +3,5 @@
     <xacro:arg name="initial_positions_file" default="initial_positions.yaml" />
     <!-- Import rtop urdf file -->
-    <xacro:include filename="$(find rtop_description)/urdf/rtop_wo_cams.urdf" />
+    <xacro:include filename="$(find rtop_description)/urdf/rtop.urdf" />
     <!-- Import control_xacro -->
     <xacro:include filename="rtop_calib.ros2_control.xacro" />

Commit message: rtop and single yam fully tested in isaac/gazebo

File: i2rt/bimanual/rtop_description/urdf/rtop.urdf (robot description, URDF)
Before this commit: robot rtop, 49 links, 48 joints
Joints:
- joint left_joint2: limit lower=0.0 upper=3.66519 effort=100 velocity=100 -> lower=-1.0e-03 upper=3.66519 effort=300 velocity=100
- joint left_joint3: limit lower=0.0 upper=3.66519 effort=100 velocity=100 -> lower=-1.0e-03 upper=3.66519 effort=300 velocity=100
- joint right_joint2: limit lower=0.0 upper=3.66519 effort=100 velocity=100 -> lower=-1.0e-03 upper=3.66519 effort=300 velocity=100
- joint right_joint3: limit lower=0.0 upper=3.66519 effort=100 velocity=100 -> lower=-1.0e-03 upper=3.66519 effort=300 velocity=100

File: i2rt/single/yam_arm_description/urdf/yam.urdf (robot description, URDF)
Before this commit: robot yam, 22 links, 21 joints
Links:
- added link camera_support, mass 0.1; collision mesh filename=package://yam_arm_description/meshes/camera_support.stl; visual mesh filename=package://yam_arm_description/meshes/camera_support.stl
- added link d435, mass 0.072; collision mesh filename=package://yam_arm_description/meshes/D435.obj; visual mesh filename=package://yam_arm_description/meshes/D435.obj
Joints:
- removed joint world2arm_fixed
- added joint camera_support2d435_fixed: type fixed, parent camera_support, child d435, origin xyz=-0.03014 0.00604 0.06023 rpy=2.6180 0.0 -1.5708
- added joint link_6_to_camera_support_fixed: type fixed, parent link_6, child camera_support, origin xyz=-0.02618 0.04089 0.05052 rpy=1.5708 1.5708 3.14159
- added joint parent2arm_fixed: type fixed, parent world, child arm, origin xyz=0.0 0.0 0.0 rpy=0.0 0.0 0.0

File: i2rt/single/yam_arm_description/urdf/yam_cam.urdf (robot description, URDF)
Before this commit: robot yam, 24 links, 23 joints
Joints:
- removed joint world2arm_fixed
- added joint parent2arm_fixed: type fixed, parent world, child arm, origin xyz=0.0 0.0 0.0 rpy=0.0 0.0 0.0

File: i2rt/single/yam_arm_moveit_config/config/yam_calib.urdf.xacro (robot description, xacro)
@@ -3,5 +3,5 @@
     <xacro:arg name="initial_positions_file" default="initial_positions.yaml" />
     <!-- Import yam_calib urdf file -->
-    <xacro:include filename="$(find yam_arm_description)/urdf/yam.urdf.xacro" />
+    <xacro:include filename="$(find yam_arm_description)/urdf/yam_cam.urdf.xacro" />
     <!-- Import control_xacro -->
     <xacro:include filename="yam_calib.ros2_control.xacro" />

Commit message: update rtop urdf with gripper mimic

File: i2rt/bimanual/rtop_description/urdf/rtop.urdf (robot description, URDF)
Before this commit: robot rtop, 49 links, 48 joints
Joints:
- joint left_right_finger: mimic (none) -> joint=left_left_finger multiplier=-1 offset=0
- joint right_right_finger: mimic (none) -> joint=right_left_finger multiplier=-1 offset=0
