Commit message: fixing urdfs, moveit assistant, usd cams

File: i2rt/single/yam_arm_moveit_config/config/yam_calib.urdf.xacro (robot description, xacro)
@@ -3,5 +3,5 @@
     <xacro:arg name="initial_positions_file" default="initial_positions.yaml" />
     <!-- Import yam_calib urdf file -->
-    <xacro:include filename="$(find yam_arm_description)/urdf/yam_cam.urdf.xacro" />
+    <xacro:include filename="$(find yam_arm_description)/urdf/yam_cam.urdf" />
     <!-- Import control_xacro -->
     <xacro:include filename="yam_calib.ros2_control.xacro" />

Commit message: fixing arm macro, rtop srdf

File: i2rt/bimanual/rtop_description/urdf/rtop.urdf (robot description, URDF)
Before this commit: robot rtop, 49 links, 48 joints
Links:
- link left_arm: geometry collision mesh filename=package://yam_arm_description/meshes/converted_model2_80808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; visual mesh filename=package://yam_arm_description/meshes/converted_model2_80808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
- link left_link_1: geometry collision mesh filename=package://yam_arm_description/meshes/converted_model2__2_80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; visual mesh filename=package://yam_arm_description/meshes/converted_model2__2_80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
- link left_link_2: geometry collision mesh filename=package://yam_arm_description/meshes/converted_model2__3_80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; collision mesh filename=package://yam_arm_description/meshes/converted_model2__4_80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
- link left_link_3: geometry collision mesh filename=package://yam_arm_description/meshes/converted_model2__6_80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; collision mesh filename=package://yam_arm_description/meshes/converted_model2__7_80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
- link left_link_4: geometry collision mesh filename=package://yam_arm_description/meshes/converted_model2__10_8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; visual mesh filename=package://yam_arm_description/meshes/converted_model2__10_8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
- link left_link_5: geometry collision mesh filename=package://yam_arm_description/meshes/converted_model2__11_8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; visual mesh filename=package://yam_arm_description/meshes/converted_model2__11_8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
- link left_link_6: geometry collision mesh filename=package://yam_arm_description/meshes/converted_model2__12_8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; collision mesh filename=package://yam_arm_description/meshes/converted_model2__13_8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
- link left_link_left_finger: geometry collision mesh filename=package://yam_arm_description/meshes/converted_model2__14_8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; collision mesh filename=package://yam_arm_description/meshes/converted_model2__15_8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
- link left_link_right_finger: geometry collision mesh filename=package://yam_arm_description/meshes/converted_model2__16_8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; collision mesh filename=package://yam_arm_description/meshes/converted_model2__17_8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
- link right_arm: geometry collision mesh filename=package://yam_arm_description/meshes/converted_model2_80808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; visual mesh filename=package://yam_arm_description/meshes/converted_model2_80808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
- link right_link_1: geometry collision mesh filename=package://yam_arm_description/meshes/converted_model2__2_80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; visual mesh filename=package://yam_arm_description/meshes/converted_model2__2_80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
- link right_link_2: geometry collision mesh filename=package://yam_arm_description/meshes/converted_model2__3_80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; collision mesh filename=package://yam_arm_description/meshes/converted_model2__4_80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
- link right_link_3: geometry collision mesh filename=package://yam_arm_description/meshes/converted_model2__6_80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; collision mesh filename=package://yam_arm_description/meshes/converted_model2__7_80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
- link right_link_4: geometry collision mesh filename=package://yam_arm_description/meshes/converted_model2__10_8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; visual mesh filename=package://yam_arm_description/meshes/converted_model2__10_8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
- link right_link_5: geometry collision mesh filename=package://yam_arm_description/meshes/converted_model2__11_8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; visual mesh filename=package://yam_arm_description/meshes/converted_model2__11_8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
- link right_link_6: geometry collision mesh filename=package://yam_arm_description/meshes/converted_model2__12_8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; collision mesh filename=package://yam_arm_description/meshes/converted_model2__13_8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
- link right_link_left_finger: geometry collision mesh filename=package://yam_arm_description/meshes/converted_model2__14_8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; collision mesh filename=package://yam_arm_description/meshes/converted_model2__15_8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
- link right_link_right_finger: geometry collision mesh filename=package://yam_arm_description/meshes/converted_model2__16_8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; collision mesh filename=package://yam_arm_description/meshes/converted_model2__17_8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

File: i2rt/bimanual/rtop_description/urdf/rtop.urdf.xacro (robot description, xacro)
@@ -68,5 +68,6 @@
     parent_link="base"
     xyz="0.0 0.305 1.0"
-    rpy="0.0 0.0 0.0"/>
+    rpy="0.0 0.0 0.0"
+    use_camera="true"/>
   <!-- Right arm: positioned at +0.305m (half of 0.610m spacing), 1m above base -->
   <xacro:yam_arm
@@ -74,4 +75,5 @@
     parent_link="base"
     xyz="0.0 -0.305 1.0"
-    rpy="0.0 0.0 0.0"/>
+    rpy="0.0 0.0 0.0"
+    use_camera="true"/>
 </robot>

File: i2rt/single/yam_arm_description/urdf/yam.urdf.xacro (robot description, xacro)
@@ -11,5 +11,5 @@
       </inertial>
    </link>
-   <!-- Use the yam_arm macro with empty prefix and parent_link="world" -->
-   <xacro:yam_arm prefix="" parent_link="world" xyz="0.0 0.0 0.0" rpy="0.0 0.0 0.0"/>
+   <!-- Use the yam_arm macro with empty prefix, parent_link="world", and camera disabled -->
+   <xacro:yam_arm prefix="" parent_link="world" xyz="0.0 0.0 0.0" rpy="0.0 0.0 0.0" use_camera="false"/>
 </robot>

File: i2rt/single/yam_arm_description/urdf/yam_arm_macro.xacro (robot description, xacro)
@@ -1,5 +1,5 @@
 <?xml version="1.0"?>
 <robot xmlns:xacro="http://www.ros.org/wiki/xacro">
-  <!-- Macro for a single YAM arm with camera (with collision meshes)
+  <!-- Macro for a single YAM arm with optional camera (with collision meshes)
        Parameters:
        - prefix: prefix for all link/joint names (e.g., "left_", "right_", or "" for no prefix)
@@ -7,6 +7,7 @@
        - xyz: position offset from parent_link
        - rpy: rotation offset from parent_link
+       - use_camera: whether to include camera components (default: false)
   -->
-  <xacro:macro name="yam_arm" params="prefix parent_link xyz rpy">
+  <xacro:macro name="yam_arm" params="prefix parent_link xyz rpy use_camera:=false">
     <!-- Arm base link -->
     <link name="${prefix}arm">
@@ -491,4 +492,55 @@
       <origin xyz="0.044 0.0 0.0" rpy="0.0 0.0 0.0"/>
     </joint>
+    <!-- Camera Support and D435 Camera (optional) -->
+    <xacro:if value="${use_camera}">
+      <link name="${prefix}camera_support">
+        <inertial>
+          <origin xyz="0.0 0.0 0.0" rpy="0.0 0.0 0.0"/>
+          <mass value="0.1"/>
+          <inertia ixx="0.0001" iyy="0.0001" izz="0.0001" ixy="0" ixz="0" iyz="0"/>
+        </inertial>
+        <visual name="${prefix}camera_support_visual">
+          <origin xyz="0.0 0.0 0.0" rpy="0.0 0.0 0.0"/>
+          <geometry>
+            <mesh filename="package://yam_arm_description/meshes/camera_support.stl"/>
+          </geometry>
+        </visual>
+        <collision name="${prefix}camera_support_collision">
+          <origin xyz="0.0 0.0 0.0" rpy="0.0 0.0 0.0"/>
+          <geometry>
+            <mesh filename="package://yam_arm_description/meshes/camera_support.stl"/>
+          </geometry>
+        </collision>
+      </link>
+      <joint type="fixed" name="${prefix}link_6_to_camera_support_fixed">
+        <parent link="${prefix}link_6"/>
+        <child link="${prefix}camera_support"/>
+        <origin xyz="-0.02618 0.04089 0.05052" rpy="1.5708 1.5708 3.14159"/>
+      </joint>
+      <link name="${prefix}d435">
+        <inertial>
+          <origin xyz="0.0 0.0 0.0" rpy="0.0 0.0 0.0"/>
+          <mass value="0.072"/>
+          <inertia ixx="0.0001" iyy="0.0001" izz="0.0001" ixy="0" ixz="0" iyz="0"/>
+        </inertial>
+        <visual name="${prefix}d435_visual">
+          <origin xyz="0.0 0.0 0.0" rpy="0.0 0.0 0.0"/>
+          <geometry>
+            <mesh filename="package://yam_arm_description/meshes/D435.obj"/>
+          </geometry>
+        </visual>
+        <collision name="${prefix}d435_collision">
+          <origin xyz="0.0 0.0 0.0" rpy="0.0 0.0 0.0"/>
+          <geometry>
+            <mesh filename="package://yam_arm_description/meshes/D435.obj"/>
+          </geometry>
+        </collision>
+      </link>
+      <joint type="fixed" name="${prefix}camera_support2d435_fixed">
+        <parent link="${prefix}camera_support"/>
+        <child link="${prefix}d435"/>
+        <origin xyz="-0.03014 0.00604 0.06023" rpy="2.6180 0.0 -1.5708"/>
+      </joint>
+    </xacro:if>
   </xacro:macro>
 </robot>

File: i2rt/single/yam_arm_description/urdf/yam_cam.urdf.xacro (robot description, xacro)
@@ -11,56 +11,5 @@
       </inertial>
    </link>
-   <!-- Use the yam_arm macro with empty prefix and parent_link="world" -->
-   <xacro:yam_arm prefix="" parent_link="world" xyz="0.0 0.0 0.0" rpy="0.0 0.0 0.0"/>
-   <!-- Camera macro (optional, for backward compatibility) -->
-   <xacro:macro name="yam_camera">
-      <link name="camera_support">
-         <inertial>
-            <origin xyz="0.0 0.0 0.0" rpy="0.0 0.0 0.0"/>
-            <mass value="0.1"/>
-            <inertia ixx="0.0001" iyy="0.0001" izz="0.0001" ixy="0" ixz="0" iyz="0"/>
-         </inertial>
-         <visual name="camera_support_visual">
-            <origin xyz="0.0 0.0 0.0" rpy="0.0 0.0 0.0"/>
-            <geometry>
-               <mesh filename="package://yam_arm_description/meshes/camera_support.stl"/>
-            </geometry>
-         </visual>
-         <collision name="camera_support_collision">
-            <origin xyz="0.0 0.0 0.0" rpy="0.0 0.0 0.0"/>
-            <geometry>
-               <mesh filename="package://yam_arm_description/meshes/camera_support.stl"/>
-            </geometry>
-         </collision>
-      </link>
-      <joint type="fixed" name="link_6_to_camera_support_fixed">
-         <parent link="link_6"/>
-         <child link="camera_support"/>
-         <origin xyz="-0.02618 0.04089 0.05052" rpy="1.5708 1.5708 3.14159"/>
-      </joint>
-      <link name="d435">
-         <inertial>
-            <origin xyz="0.0 0.0 0.0" rpy="0.0 0.0 0.0"/>
-            <mass value="0.072"/>
-            <inertia ixx="0.0001" iyy="0.0001" izz="0.0001" ixy="0" ixz="0" iyz="0"/>
-         </inertial>
-         <visual name="d435_visual">
-            <origin xyz="0.0 0.0 0.0" rpy="0.0 0.0 0.0"/>
-            <geometry>
-               <mesh filename="package://yam_arm_description/meshes/D435.obj"/>
-            </geometry>
-         </visual>
-         <collision name="d435_collision">
-            <origin xyz="0.0 0.0 0.0" rpy="0.0 0.0 0.0"/>
-            <geometry>
-               <mesh filename="package://yam_arm_description/meshes/D435.obj"/>
-            </geometry>
-         </collision>
-      </link>
-      <joint type="fixed" name="camera_support2d435_fixed">
-         <parent link="camera_support"/>
-         <child link="d435"/>
-         <origin xyz="-0.03014 0.00604 0.06023" rpy="2.6180 0.0 -1.5708"/>
-      </joint>
-   </xacro:macro>
+   <!-- Use the yam_arm macro with empty prefix, parent_link="world", and camera enabled -->
+   <xacro:yam_arm prefix="" parent_link="world" xyz="0.0 0.0 0.0" rpy="0.0 0.0 0.0" use_camera="true"/>
 </robot>
