Commit message: gazebo, single arm working in gazebo

File: i2rt/bimanual/rtop_moveit_config/config/rtop_calib.urdf.xacro (robot description, xacro)
@@ -1,4 +1,4 @@
 <?xml version="1.0"?>
-<robot xmlns:xacro="http://www.ros.org/wiki/xacro" name="rtop_calib">
+<robot xmlns:xacro="http://www.ros.org/wiki/xacro" name="rtop">
     <xacro:arg name="initial_positions_file" default="initial_positions.yaml" />
     <!-- Import rtop urdf file -->

File: i2rt/single/yam_arm_description/urdf/yam.urdf.xacro (robot description, xacro)
@@ -96,5 +96,5 @@
       <origin xyz="2.5e-05 -0.02 0.0409" rpy="1.5707963267948966 0.0 1.5707963267948966"/>
       <axis xyz="0.0 0.0 1.0"/>
-      <limit lower="-3.66519" upper="3.66519" effort="300" velocity="100"/>
+      <limit lower="-1.0e-03" upper="3.66519" effort="300" velocity="100"/>
    </joint>
    <joint type="fixed" name="joint2_offset">
@@ -146,5 +146,5 @@
       <origin xyz="0.264 0.0 0.0" rpy="3.141592653589793 0.0 0.0"/>
       <axis xyz="0.0 0.0 1.0"/>
-      <limit lower="-3.66519" upper="3.66519" effort="300" velocity="100"/>
+      <limit lower="-1.0e-03" upper="3.66519" effort="300" velocity="100"/>
    </joint>
    <joint type="fixed" name="joint3_offset">

File: i2rt/single/yam_arm_description/urdf/yam_cam.urdf (robot description, URDF)
Before this commit: robot yam, 24 links, 23 joints
Links:
- removed link joint1
- removed link joint2
- removed link joint3
- removed link joint4
- removed link joint5
- removed link joint6
- removed link left_finger
- removed link right_finger
- added link joint1_link, mass 0.001
- added link joint2_link, mass 0.001
- added link joint3_link, mass 0.001
- added link joint4_link, mass 0.001
- added link joint5_link, mass 0.001
- added link joint6_link, mass 0.001
- added link left_finger_link, mass 0.001
- added link right_finger_link, mass 0.001
Joints:
- joint joint1: child joint1 -> joint1_link
- joint joint1_offset: parent joint1 -> joint1_link
- joint joint2: child joint2 -> joint2_link
- joint joint2_offset: parent joint2 -> joint2_link
- joint joint3: child joint3 -> joint3_link
- joint joint3_offset: parent joint3 -> joint3_link
- joint joint4: child joint4 -> joint4_link
- joint joint4_offset: parent joint4 -> joint4_link
- joint joint5: child joint5 -> joint5_link
- joint joint5_offset: parent joint5 -> joint5_link
- joint joint6: child joint6 -> joint6_link
- joint joint6_offset: parent joint6 -> joint6_link
- joint left_finger: child left_finger -> left_finger_link
- joint left_finger_offset: parent left_finger -> left_finger_link
- joint right_finger: child right_finger -> right_finger_link
- joint right_finger_offset: parent right_finger -> right_finger_link

File: i2rt/single/yam_arm_moveit_config/config/yam_calib.urdf.xacro (robot description, xacro)
@@ -3,5 +3,5 @@
     <xacro:arg name="initial_positions_file" default="initial_positions.yaml" />
     <!-- Import yam_calib urdf file -->
-    <xacro:include filename="$(find yam_arm_description)/urdf/yam.urdf" />
+    <xacro:include filename="$(find yam_arm_description)/urdf/yam.urdf.xacro" />
     <!-- Import control_xacro -->
     <xacro:include filename="yam_calib.ros2_control.xacro" />
