Commit message: jazzy left arm and gripper working, right is not

File: i2rt/bimanual/rtop_moveit_config/config/rtop_calib.ros2_control.xacro (robot description, xacro)
@@ -2,11 +2,11 @@
 <robot xmlns:xacro="http://www.ros.org/wiki/xacro">
     <xacro:macro name="rtop_calib_ros2_control" params="name initial_positions_file">
-        <xacro:property name="initial_positions" value="${load_yaml(initial_positions_file)['initial_positions']}"/>
+        <xacro:property name="initial_positions" value="${xacro.load_yaml(initial_positions_file)['initial_positions']}"/>
         <ros2_control name="${name}" type="system">
             <hardware>
-                <!-- By default, set up controllers for simulation. This won't work on real hardware -->
-                <!-- plugin>mock_components/GenericSystem</plugin -->
+                <!-- For Isaac Sim: use topic_based_ros2_control to interface via topics -->
+                <!-- This plugin reads joint_states from /joint_states and writes commands to /joint_command -->
                 <plugin>topic_based_ros2_control/TopicBasedSystem</plugin>
-                <param name="joint_commands_topic">/joint_command</param>
+                <param name="joint_commands_topic">/joint_command_raw</param>
                 <param name="joint_states_topic">/joint_states</param>
             </hardware>
@@ -61,5 +61,5 @@
                 <state_interface name="velocity"/>
             </joint>
-            <!-- left_right_finger: mimic joint (no command interface for Jazzy compatibility) -->
+            <!-- left_right_finger: mimic joint (no command interface - mimic joints cannot have command interfaces) -->
             <joint name="left_right_finger">
                 <state_interface name="position">
@@ -118,5 +118,5 @@
                 <state_interface name="velocity"/>
             </joint>
-            <!-- right_right_finger: mimic joint (no command interface for Jazzy compatibility) -->
+            <!-- right_right_finger: mimic joint (no command interface - mimic joints cannot have command interfaces) -->
             <joint name="right_right_finger">
                 <state_interface name="position">
