Commit message: ctrl gz working single, moveit some pos are not working, reorder code

File: i2rt/single/yam_arm_description/urdf/yam.urdf (robot description, URDF)
Before this commit: robot yam, 22 links, 21 joints
Joints:
- joint joint2: limit lower=-3.66519 upper=3.66519 effort=300 velocity=100 -> lower=-1.0e-03 upper=3.66519 effort=300 velocity=100
- joint joint3: limit lower=-3.66519 upper=3.66519 effort=300 velocity=100 -> lower=-1.0e-03 upper=3.66519 effort=300 velocity=100

File: i2rt/single/yam_arm_description/urdf/yam.urdf.xacro (robot description, xacro)
@@ -379,3 +379,54 @@
       <origin xyz="0.044 0.0 0.0" rpy="0.0 0.0 0.0"/>
    </joint>
+   <!-- Camera macro (optional) -->
+   <xacro:macro name="yam_camera">
+      <link name="camera_support">
+         <inertial>
+            <origin xyz="0.0 0.0 0.0" rpy="0.0 0.0 0.0"/>
+            <mass value="0.1"/>
+            <inertia ixx="0.0001" iyy="0.0001" izz="0.0001" ixy="0" ixz="0" iyz="0"/>
+         </inertial>
+         <visual name="camera_support_visual">
+            <origin xyz="0.0 0.0 0.0" rpy="0.0 0.0 0.0"/>
+            <geometry>
+               <mesh filename="package://yam_arm_description/meshes/camera_support.stl"/>
+            </geometry>
+         </visual>
+         <collision name="camera_support_collision">
+            <origin xyz="0.0 0.0 0.0" rpy="0.0 0.0 0.0"/>
+            <geometry>
+               <mesh filename="package://yam_arm_description/meshes/camera_support.stl"/>
+            </geometry>
+         </collision>
+      </link>
+      <joint type="fixed" name="link_6_to_camera_support_fixed">
+         <parent link="link_6"/>
+         <child link="camera_support"/>
+         <origin xyz="-0.02618 0.04089 0.05052" rpy="1.5708 1.5708 3.14159"/>
+      </joint>
+      <link name="d435">
+         <inertial>
+            <origin xyz="0.0 0.0 0.0" rpy="0.0 0.0 0.0"/>
+            <mass value="0.072"/>
+            <inertia ixx="0.0001" iyy="0.0001" izz="0.0001" ixy="0" ixz="0" iyz="0"/>
+         </inertial>
+         <visual name="d435_visual">
+            <origin xyz="0.0 0.0 0.0" rpy="0.0 0.0 0.0"/>
+            <geometry>
+               <mesh filename="package://yam_arm_description/meshes/D435.obj"/>
+            </geometry>
+         </visual>
+         <collision name="d435_collision">
+            <origin xyz="0.0 0.0 0.0" rpy="0.0 0.0 0.0"/>
+            <geometry>
+               <mesh filename="package://yam_arm_description/meshes/D435.obj"/>
+            </geometry>
+         </collision>
+      </link>
+      <joint type="fixed" name="camera_support2d435_fixed">
+         <parent link="camera_support"/>
+         <child link="d435"/>
+         <origin xyz="-0.03014 0.00604 0.06023" rpy="2.6180 0.0 -1.5708"/>
+      </joint>
+   </xacro:macro>
 </robot>

File: i2rt/single/yam_arm_description/urdf/yam_arm_gazebo.urdf.xacro (robot description, xacro)
@@ -8,8 +8,67 @@
   <!-- ROS2 Control for Gazebo -->
   <xacro:if value="$(arg use_gazebo)">
-    <xacro:include filename="$(find yam_arm_description)/urdf/gazebo_sim_ros2_control.urdf.xacro"/>
-    <xacro:load_gazebo_sim_ros2_control_plugin robot_name="yam" ros2_controllers_path="$(arg ros2_controllers_path)" use_gazebo="$(arg use_gazebo)"/>
-    <xacro:include filename="$(find yam_arm_description)/urdf/ros2_control.urdf.xacro" />
-    <xacro:ros2_control_interfaces/>
+    <!-- Gazebo ROS2 Control Plugin -->
+    <gazebo>
+      <plugin filename="gz_ros2_control-system" name="gz_ros2_control::GazeboSimROS2ControlPlugin">
+        <parameters>$(arg ros2_controllers_path)</parameters>
+        <ros>
+          <remapping>/controller_manager/robot_description:=/robot_description</remapping>
+        </ros>
+      </plugin>
+    </gazebo>
+    <!-- ROS2 Control Interfaces -->
+    <ros2_control name="IgnitionSystem" type="system">
+      <hardware>
+        <plugin>gz_ros2_control/GazeboSimSystem</plugin>
+      </hardware>
+      <joint name="joint1">
+        <command_interface name="position"/>
+        <state_interface name="position" />
+        <state_interface name="velocity"/>
+        <state_interface name="effort"/>
+      </joint>
+      <joint name="joint2">
+        <command_interface name="position"/>
+        <state_interface name="position"/>
+        <state_interface name="velocity"/>
+        <state_interface name="effort"/>
+      </joint>
+      <joint name="joint3">
+        <command_interface name="position"/>
+        <state_interface name="position"/>
+        <state_interface name="velocity"/>
+        <state_interface name="effort"/>
+      </joint>
+      <joint name="joint4">
+        <command_interface name="position"/>
+        <state_interface name="position"/>
+        <state_interface name="velocity"/>
+        <state_interface name="effort"/>
+      </joint>
+      <joint name="joint5">
+        <command_interface name="position"/>
+        <state_interface name="position"/>
+        <state_interface name="velocity"/>
+        <state_interface name="effort"/>
+      </joint>
+      <joint name="joint6">
+        <command_interface name="position"/>
+        <state_interface name="position"/>
+        <state_interface name="velocity"/>
+        <state_interface name="effort"/>
+      </joint>
+      <joint name="left_finger">
+        <command_interface name="position"/>
+        <state_interface name="position"/>
+        <state_interface name="velocity"/>
+        <state_interface name="effort"/>
+      </joint>
+      <joint name="right_finger">
+        <command_interface name="position"/>
+        <state_interface name="position"/>
+        <state_interface name="velocity"/>
+        <state_interface name="effort"/>
+      </joint>
+    </ros2_control>
   </xacro:if>
 </robot>

File: i2rt/single/yam_arm_description/urdf/yam_cam.urdf (robot description, URDF)
Before this commit: robot yam, 24 links, 23 joints
Joints:
- joint joint2: limit lower=0.0 upper=3.66519 effort=100 velocity=100 -> lower=-1.0e-03 upper=3.66519 effort=300 velocity=100
- joint joint3: limit lower=0.0 upper=3.66519 effort=100 velocity=100 -> lower=-1.0e-03 upper=3.66519 effort=300 velocity=100
