Commit message: yam arm camera support color works, but other links nope

File: i2rt/single/yam_arm_description/urdf/yam_arm_gazebo.urdf.xacro (robot description, xacro)
@@ -16,4 +16,15 @@
         </ros>
       </plugin>
+    </gazebo>
+    <!-- Gazebo Material Colors for Links using RGBA values -->
+    <!-- Camera -->
+    <gazebo reference="camera_support">
+      <visual>
+        <material>
+          <ambient>0.1 0.1 0.1 1.0</ambient>
+          <diffuse>0.1 0.1 0.1 1.0</diffuse>
+          <specular>0.1 0.1 0.1 1.0</specular>
+        </material>
+      </visual>
     </gazebo>
     <!-- ROS2 Control Interfaces -->
