Commit message: gripper mimic working

File: i2rt/single/yam_arm_description/urdf/yam_arm_macro.xacro (robot description, xacro)
@@ -358,4 +358,5 @@
       <axis xyz="0.0 0.0 1.0"/>
       <limit lower="-0.037524" upper="0.00205" effort="100" velocity="100"/>
+      <mimic joint="${prefix}left_finger" multiplier="-1" offset="0"/>
     </joint>
     <joint type="fixed" name="${prefix}right_finger_offset">

File: i2rt/single/yam_arm_description/urdf/yam_cam.urdf (robot description, URDF)
Before this commit: robot yam, 24 links, 23 joints
Joints:
- joint right_finger: mimic (none) -> joint=left_finger multiplier=-1 offset=0

File: i2rt/single/yam_arm_moveit_config/config/yam_calib.ros2_control.xacro (robot description, xacro)
@@ -8,6 +8,6 @@
                 <!-- plugin>mock_components/GenericSystem</plugin -->
                 <plugin>topic_based_ros2_control/TopicBasedSystem</plugin>
-                <param name="joint_commands_topic">/isaac_joint_command</param>
-                <param name="joint_states_topic">/isaac_joint_states</param>
+                <param name="joint_commands_topic">/joint_command</param>
+                <param name="joint_states_topic">/joint_states</param>
             </hardware>
             <joint name="joint1">
@@ -61,4 +61,6 @@
             </joint>
             <joint name="right_finger">
+                <!-- Command interface kept for Isaac Sim compatibility (expects 8 values) -->
+                <!-- Actual control handled by URDF mimic joint - no controller uses this -->
                 <command_interface name="position"/>
                 <state_interface name="position">

File: i2rt/single/yam_arm_moveit_config/config/yam_calib.urdf.xacro (robot description, xacro)
@@ -1,4 +1,4 @@
 <?xml version="1.0"?>
-<robot xmlns:xacro="http://www.ros.org/wiki/xacro" name="yam_calib">
+<robot xmlns:xacro="http://www.ros.org/wiki/xacro" name="yam">
     <xacro:arg name="initial_positions_file" default="initial_positions.yaml" />
     <!-- Import yam_calib urdf file -->
